File: hardware/ledcontroller_3x/ledcontroller.kicad_pcb (KiCad board)
At the start: 4 copper layers, 38 x 59 mm, 90 parts, among them J13 TX, J14 RX, J15 FLASH, J16 SCL, J17 SDA, J18 OE, J19 Pololu D24V5F3, J2 GPIO16, J20 VIN, J21 GND, J22 24V, J23 RED, J24 GREEN, J25 BLUE, J26 W_WHITE, J27 C_WHITE, J28 24V, J29 RED, J30 GREEN, J31 BLUE, J32 W_WHITE, J33 C_WHITE, J34 24V, J35 RED, J36 GREEN, J37 BLUE, J38 W_WHITE, J39 C_WHITE, J41 Flash Adapter, J6 RESET, Q1 BLM3400, Q10 BLM3400, Q11 BLM3400, Q12 BLM3400, Q13 BLM3400, Q14 BLM3400, Q15 BLM3400, Q16 MMS9013-H-TP, Q17 MMS9013-H-TP, Q2 BLM3400, Q3 BLM3400, Q4 BLM3400, Q5 BLM3400, Q6 BLM3400, Q7 BLM3400, Q8 BLM3400, Q9 BLM3400, U1 ESP-12E, U2 PCA9685PW

Commit message: fixed typo in silkscreen
Other:
- board text added: "DTR"
- board text removed: "DRT"
Changed lines of the file:
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@@
     (effects (font (size 1 1) (thickness 0.15)) (justify mirror))
   )
-  (gr_text "DRT" (at 123.19 81.28) (layer "B.SilkS")
+  (gr_text "DTR" (at 123.19 81.28) (layer "B.SilkS")
     (effects (font (size 1 1) (thickness 0.15)) (justify left bottom mirror))
   )
